File: HITLBoardV0P1/Ethernet.kicad_sch (KiCad schematic)
At the start: 16 parts, among them U2 LAN8650B1-E/LMX, U3 LP38852MRX-ADJ/NOPB

Commit message: complete ethernet schematic capture
Parts:
- added C10, C11, C12, C9: 10u, Capacitor_SMD:C_0402_1005Metric, symbol Device:C
- added C13, C15, C17, C19, C21: 10n, Capacitor_SMD:C_0402_1005Metric, symbol Device:C
- added C14, C16, C18, C20, C22, C23, C24, C25: .1U, Capacitor_SMD:C_0402_1005Metric, symbol Device:C
- added R6, R7: 49.9K, Resistor_SMD:R_0402_1005Metric, symbol Device:R_US
- added R8: 100K, Resistor_SMD:R_0402_1005Metric, symbol Device:R_US
Connections:
- net +3V3: now also C10.1, C11.1, C12.1, C13.1, C14.1, C15.1, C16.1, C17.1, C18.1, C19.1, C20.1, C21.1, C22.1, C9.1
- net GND: now also C10.2, C11.2, C12.2, C13.2, C14.2, C15.2, C16.2, C17.2, C18.2, C19.2, C20.2, C21.2, C22.2, C25.1, C9.2, R8.2
- net TRXP: now reaches U2.30 (TRXP)
- net TRXP: now also C24.1
- net TRXN: now reaches U2.31 (TRXN)
- net TRXN: now also C23.1
- new net: C25.2, R6.2, R7.2, R8.1
- new net ETH_10T1S_TRXN: C23.2, R7.1
- new net ETH_10T1S_TRXP: C24.2, R6.1
Other:
- note added: "PIN 15"
- note added: "PIN 17"
- note added: "PIN 21"
- note added: "PIN 6"
- note added: "PIN 7"
- note added: "PLACE 10 NF CLOSEST TO PIN (TYPICAL)"
- moved on the sheet: C1, C2, C3, C4, C5, U3
