File: HITLBoardV0P1/Ethernet2.kicad_sch (KiCad schematic)
At the start: 36 parts, among them U2 LAN8650B1-E/LMX, U3 LP38852MRX-ADJ/NOPB

Commit message: UPDATE -- IN PROGRESS
Parts:
- renumbered C10 to C26, C11 to C27, C9 to C28, C12 to C29, C13 to C30, C15 to C31, C17 to C32, C14 to C33, C16 to C34, C18 to C35, C6 to C36, C7 to C37, C19 to C38, C21 to C39, C8 to C40, C20 to C41, C22 to C42, C4 to C43, C3 to C44, C23 to C45, C24 to C46, C5 to C47, C25 to C48, C1 to C49, C2 to C50, R4 to R10, R5 to R11, R1 to R12, R2 to R13, R6 to R14, R7 to R15, R8 to R16, R3 to R9, U2 to U4, U3 to U5, XTAL1 to XTAL2
Connections:
- net +3V3: now also C30.1, C31.1, C32.1, C33.1, C34.1, C35.1
- net 1V8_U2: no longer C30.1, C31.1, C32.1, C33.1, C34.1, C35.1
- net GND: no longer U5.9 (DAP)
- net ETH_10T1S_TRXN_N renamed ETH_10T1S_TRXN
- net ETH_10T1S_TRXP_P renamed ETH_10T1S_TRXP
- net TRXN_N renamed TRXN
- net TRXP_P renamed TRXP
- new net U3_DAP: U5.9 (DAP)
- no-connect marks 3 -> 2
Other:
- moved on the sheet: C26, C27, C28, C29, C30, C31, C32, C33, C34, C35, C36, C37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

Commit message: in progress, brute forced lan8650 layouts :( damn you kicad
Connections:
- net +3V3: no longer C30.1, C31.1, C32.1, C33.1, C34.1, C35.1
- net 1V8_U2 renamed 1V8
- net 1V8: now also C30.1, C31.1, C32.1, C33.1, C34.1, C35.1
Other:
- moved on the sheet: C26, C27, C28, C29, C30, C31, C32, C33, C34, C35, C36, C37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

Commit message: MINOR UPDATES -- SWTICH ONE LAN TO SPI 5 INSTEAD OF SPI1 ON THE TMDX, SET UP LAN8650S for actual differential pair routing by changing suffix to "_DN" and "_DP" instead of "_N" or "_P" or just "N", "P"
Connections:
- net TRXN renamed TRX_DN
- net TRXP renamed TRX_DP
Changed lines of the file:
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@@
 		)
 	)
-	(label "TRXP"
+	(label "TRX_DP"
 		(at 99.06 67.31 0)
 		(effects
@@
 		)
 	)
-	(label "ETH_10T1S_TRXN"
+	(label "ETH_10T1S_TRX_DN"
 		(at 334.01 50.8 0)
 		(effects
@@
 		)
 	)
-	(label "TRXN"
+	(label "TRX_DN"
 		(at 99.06 64.77 0)
 		(effects
@@
 		)
 	)
-	(label "TRXN"
+	(label "TRX_DN"
 		(at 298.45 50.8 0)
 		(effects
@@
 		)
 	)
-	(label "ETH_10T1S_TRXP"
+	(label "ETH_10T1S_TRX_DP"
 		(at 334.01 58.42 0)
 		(effects
@@
 		)
 	)
-	(label "TRXP"
+	(label "TRX_DP"
 		(at 298.45 91.44 0)
 		(effects
