File: HITLBoardV0P1/ethernet3.kicad_sch (KiCad schematic)
At the start: 36 parts, among them U2 LAN8650B1-E/LMX, U3 LP38852MRX-ADJ/NOPB

Commit message: in progress, brute forced lan8650 layouts :( damn you kicad
Parts:
- renumbered C1 to C51, C2 to C52, C3 to C53, C4 to C54, C5 to C55, C6 to C56, C7 to C57, C8 to C58, C9 to C59, C10 to C60, C11 to C61, C12 to C62, C13 to C63, C14 to C64, C15 to C65, C16 to C66, C17 to C67, C18 to C68, C19 to C69, C20 to C70, C21 to C71, C22 to C72, C23 to C73, C24 to C74, C25 to C75, R1 to R17, R2 to R18, R3 to R19, R4 to R20, R5 to R21, R6 to R22, R7 to R23, R8 to R24, U2 to U6, U3 to U7, XTAL1 to XTAL3
Connections:
- net U3_DAP is gone; now on net GND: U7.9 (DAP)
- net +3V3: no longer C55.1, C56.1, C57.1, C58.1, C59.1, C60.1
- net 1V8_U2 renamed 1V8
- net 1V8: now also C55.1, C56.1, C57.1, C58.1, C59.1, C60.1
Other:
- moved on the sheet: C51, C52, C53, C54, C55, C56, C57, C58, C59, C60, C61, C62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

Commit message: MINOR UPDATES -- SWTICH ONE LAN TO SPI 5 INSTEAD OF SPI1 ON THE TMDX, SET UP LAN8650S for actual differential pair routing by changing suffix to "_DN" and "_DP" instead of "_N" or "_P" or just "N", "P"
Connections:
- net TRXN renamed TRX_DN
- net TRXP renamed TRX_DP
Changed lines of the file:
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@@
 		)
 	)
-	(label "TRXP"
+	(label "TRX_DP"
 		(at 106.68 52.07 0)
 		(effects
@@
 		)
 	)
-	(label "ETH_10T1S_TRXN"
+	(label "ETH_10T1S_TRX_DN"
 		(at 341.63 35.56 0)
 		(effects
@@
 		)
 	)
-	(label "TRXN"
+	(label "TRX_DN"
 		(at 106.68 49.53 0)
 		(effects
@@
 		)
 	)
-	(label "TRXN"
+	(label "TRX_DN"
 		(at 306.07 35.56 0)
 		(effects
@@
 		)
 	)
-	(label "ETH_10T1S_TRXP"
+	(label "ETH_10T1S_TRX_DP"
 		(at 341.63 43.18 0)
 		(effects
@@
 		)
 	)
-	(label "TRXP"
+	(label "TRX_DP"
 		(at 306.07 76.2 0)
 		(effects
