File: HITLBoardV0P1/I2C_GPIO_EXPANDER.kicad_sch (KiCad schematic)
At the start: 5 parts, among them U24 MCP23008-E/SO

Commit message: add debug LEDs and reset_n button for system reset
Changed lines of the file:
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@@
+		)
+	)
+	(hierarchical_label "RESET_N"
+		(shape input)
+		(at 127 115.57 180)
+		(effects
+			(font
+				(size 1.27 1.27)
+			)
+			(justify right)
 		)
 	)

Commit message: FIX spi 3 on tmdx for current loop ADC, add gpio pin for data ready
Connections:
- net A0: now reaches R68.2, U24.5 (A0)
Changed lines of the file:
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@@
+	(wire
+		(pts
+			(xy 138.43 201.93) (xy 156.21 201.93)
+		)
+		(stroke
+			(width 0)
+			(type default)
+		)
+	)
 	(wire
 		(pts
@@
 	(wire
 		(pts
+			(xy 127 113.03) (xy 146.05 113.03)
+		)
+		(stroke
+			(width 0)
+			(type default)
+		)
+	)
+	(wire
+		(pts
 			(xy 127 110.49) (xy 146.05 110.49)
 		)
@@
 	(wire
 		(pts
-			(xy 127 113.03) (xy 146.05 113.03)
-		)
-		(stroke
-			(width 0)
-			(type default)
-		)
-	)
-	(wire
-		(pts
 			(xy 214.63 97.79) (xy 214.63 102.87)
-		)
-		(stroke
-			(width 0)
-			(type default)
-		)
-	)
-	(wire
-		(pts
-			(xy 137.16 201.93) (xy 156.21 201.93)
 		)
 		(stroke
@@
 		)
 	)
+	(label "GP4"
+		(at 210.82 113.03 0)
+		(effects
+			(font
+				(size 1.27 1.27)
+			)
+			(justify left bottom)
+		)
+	)
+	(label "A1"
+		(at 143.51 184.15 0)
+		(effects
+			(font
+				(size 1.27 1.27)
+			)
+			(justify left bottom)
+		)
+	)
+	(label "GP1"
+		(at 210.82 120.65 0)
+		(effects
+			(font
+				(size 1.27 1.27)
+			)
+			(justify left bottom)
+		)
+	)
+	(label "RESET_N"
+		(at 130.81 115.57 0)
+		(effects
+			(font
+				(size 1.27 1.27)
+			)
+			(justify left bottom)
+		)
+	)
 	(label "A0"
 		(at 133.35 113.03 0)
 		(effects
-			(font
-				(size 1.27 1.27)
-			)
-			(justify left bottom)
-		)
-	)
-	(label "GP4"
-		(at 210.82 113.03 0)
-		(effects
-			(font
-				(size 1.27 1.27)
-			)
-			(justify left bottom)
-		)
-	)
-	(label "A1"
-		(at 143.51 184.15 0)
-		(effects
-			(font
-				(size 1.27 1.27)
-			)
-			(justify left bottom)
-		)
-	)
-	(label "GP1"
-		(at 210.82 120.65 0)
-		(effects
-			(font
-				(size 1.27 1.27)
-			)
-			(justify left bottom)
-		)
-	)
-	(label "RESET_N"
-		(at 130.81 115.57 0)
-		(effects
-			(font
-				(size 1.27 1.27)
-			)
-			(justify left bottom)
-		)
-	)
-	(label ""
-		(at 133.35 113.03 0)
-		(effects
