File: HITLBoardV0P1/RaspberryPiPico.kicad_sch (KiCad schematic)
At the start: 3 parts, among them J1 USB_B_Micro, J2 FTSH-105-01-L-DV

Commit message: in progress, brute forced lan8650 layouts :( damn you kicad
Parts:
- removed J1: USB_B_Micro, symbol Connector:USB_B_Micro
Connections:
- net USB_2P0_D_N: no longer names the net of A1.TP2 (USB_DM)
- net USB_2P0_D_P: no longer names the net of A1.TP3 (USB_DP)
- no-connect marks 6 -> 5

Commit message: update
Changed lines of the file:
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@@
-	)
-	(symbol
-		(lib_id "power:+3.3VP")
-		(at 186.69 71.12 0)
-		(unit 1)
-		(body_style 1)
-		(exclude_from_sim no)
-		(in_bom yes)
-		(on_board yes)
-		(in_pos_files yes)
-		(dnp no)
-		(fields_autoplaced yes)
-		(property "Reference" "#PWR0130"
-			(at 190.5 72.39 0)
-			(hide yes)
-			(show_name no)
-			(do_not_autoplace no)
-			(effects
-				(font
-					(size 1.27 1.27)
-				)
-			)
-		)
-		(property "Value" "+3.3VP"
-			(at 186.69 66.04 0)
-			(show_name no)
-			(do_not_autoplace no)
-			(effects
-				(font
-					(size 1.27 1.27)
-				)
-			)
-		)
-		(property "Footprint" ""
-			(at 186.69 71.12 0)
-			(hide yes)
-			(show_name no)
-			(do_not_autoplace no)
-			(effects
-				(font
-					(size 1.27 1.27)
-				)
-			)
-		)
-		(property "Datasheet" ""
-			(at 186.69 71.12 0)
-			(hide yes)
-			(show_name no)
-			(do_not_autoplace no)
-			(effects
-				(font
-					(size 1.27 1.27)
-				)
-			)
-		)
-		(property "Description" "Power symbol creates a global label with name \"+3.3VP\""
-			(at 186.69 71.12 0)
-			(hide yes)
-			(show_name no)
-			(do_not_autoplace no)
-			(effects
-				(font
-					(size 1.27 1.27)
-				)
-			)
-		)
-		(pin "1"
-		)
-		(instances
-			(project "HITLBoardV0P1"
-				(path "/ef043e91-6391-40b5-b326-2e3f2f5d4c07/1802981a-1ca5-49a5-8666-49bc80282853"
-					(reference "#PWR0130")
-					(unit 1)
-				)
-			)
-		)
 	)
 	(symbol

Commit message: add debug LEDs and reset_n button for system reset
Parts:
- added R84: 10K, Resistor_SMD:R_01005_0402Metric, symbol Device:R_US
- added SW2: SW_Push, Button_Switch_SMD:SW_Push_1P1T_NO_E-Switch_TL3301NxxxxxG, symbol Switch:SW_Push
Connections:
- net +3.3VP: now also R84.1
- net GND: now also SW2.2
- net BOOTSEL_N: now reaches A1.TP6 (~{BOOTSEL})
- net BOOTSEL_N: now also R84.2, SW2.1
- no-connect marks 5 -> 4

Commit message: basic organization into layout
Parts:
- removed R84: 10K, Resistor_SMD:R_01005_0402Metric, symbol Device:R_US
- removed SW2: SW_Push, Button_Switch_SMD:SW_Push_1P1T_NO_E-Switch_TL3301NxxxxxG, symbol Switch:SW_Push
